Commit message: small fix

File: src/robot_arms/descriptions/urdf/franka/fr3_franka_hand.urdf (robot description, URDF)
Before this commit: robot fr3, 13 links, 12 joints
Links:
- added link fr3_link4, mass 2.6155955791; collision mesh filename=franka_description/meshes/robot_arms/fr3/collision/link4.stl; visual mesh filename=franka_description/meshes/robot_arms/fr3/visual/link4.dae
- link fr3_link3: mass 2.6155955791 -> 2.2449013699
Joints:
- added joint fr3_joint3: type revolute, parent fr3_link2, child fr3_link3, origin xyz=0 -0.316 0 rpy=1.570796326794897 0 0, axis 0 0 1, limit lower=-2.9007 upper=2.9007 effort=87.0 velocity=2.62
